File: Servo_Power.kicad_sch (KiCad schematic)
At the start: 11 parts, among them J2 SERVO_BUCK_IN, J3 SERVO_BUCK_OUT, J4 Servo1, J5 Servo2, J6 Servo3, J7 Servo4, J8 Servo5

Commit message: BNO086 I2C connection added
Other:
- moved on the sheet: C6, C7
Changed lines of the file:
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@@
 	(paper "A4")
-	(junction
-		(at 179.07 90.17)
-		(diameter 0)
-		(color 0 0 0 0)
-	)
 	(junction
 		(at 149.86 97.79)
@@
 	)
 	(junction
-		(at 127 97.79)
+		(at 172.72 97.79)
 		(diameter 0)
 		(color 0 0 0 0)
 	)
 	(junction
-		(at 179.07 97.79)
+		(at 172.72 90.17)
+		(diameter 0)
+		(color 0 0 0 0)
+	)
+	(junction
+		(at 127 97.79)
 		(diameter 0)
 		(color 0 0 0 0)
@@
 	(wire
 		(pts
+			(xy 172.72 97.79) (xy 185.42 97.79)
+		)
+		(stroke
+			(width 0)
+			(type default)
+		)
+	)
+	(wire
+		(pts
 			(xy 87.63 90.17) (xy 96.52 90.17)
 		)
@@
 	(wire
 		(pts
-			(xy 53.34 90.17) (xy -30.48 90.17)
-		)
-		(stroke
-			(width 0)
-			(type default)
-		)
-	)
-	(wire
-		(pts
 			(xy 209.55 104.14) (xy 214.63 104.14)
 		)
@@
 	(wire
 		(pts
-			(xy 179.07 90.17) (xy 193.04 90.17)
-		)
-		(stroke
-			(width 0)
-			(type default)
-		)
-	)
-	(wire
-		(pts
 			(xy 54.61 90.17) (xy 80.01 90.17)
 		)
@@
 	(wire
 		(pts
-			(xy 179.07 97.79) (xy 193.04 97.79)
-		)
-		(stroke
-			(width 0)
-			(type default)
-		)
-	)
-	(wire
-		(pts
 			(xy 214.63 129.54) (xy 209.55 129.54)
 		)
@@
 	(wire
 		(pts
-			(xy -30.48 0.8096) (xy 0.3048 0.8096)
+			(xy -1.27 90.17) (xy 53.34 90.17)
 		)
 		(stroke
@@
 	(wire
 		(pts
-			(xy -30.48 90.17) (xy -30.48 0.8096)
-		)
-		(stroke
-			(width 0)
-			(type default)
-		)
-	)
-	(wire
-		(pts
 			(xy 133.35 90.17) (xy 149.86 90.17)
 		)
@@
 	(wire
 		(pts
+			(xy 172.72 90.17) (xy 185.42 90.17)
+		)
+		(stroke
+			(width 0)
+			(type default)
+		)
+	)
+	(wire
+		(pts
 			(xy 209.55 78.74) (xy 214.63 78.74)
 		)
@@
 	(wire
 		(pts
-			(xy 149.86 90.17) (xy 179.07 90.17)
-		)
-		(stroke
-			(width 0)
-			(type default)
-		)
-	)
-	(wire
-		(pts
-			(xy 149.86 97.79) (xy 179.07 97.79)
+			(xy 149.86 90.17) (xy 172.72 90.17)
+		)
+		(stroke
+			(width 0)
+			(type default)
+		)
+	)
+	(wire
+		(pts
+			(xy 149.86 97.79) (xy 172.72 97.79)
 		)
 		(stroke
@@
 	(symbol
 		(lib_id "Device:C")
-		(at 179.07 93.98 0)
+		(at 172.72 93.98 0)
 		(unit 1)
 		(body_style 1)
@@
 		(fields_autoplaced yes)
 		(property "Reference" "C6"
-			(at 182.88 92.7099 0)
+			(at 176.53 92.7099 0)
 			(show_name no)
 			(do_not_autoplace no)
@@
 		)
 		(property "Value" "10 µF"
-			(at 182.88 95.2499 0)
+			(at 176.53 95.2499 0)
 			(show_name no)
 			(do_not_autoplace no)
@@
 		)
 		(property "Footprint" ""
-			(at 180.0352 97.79 0)
+			(at 173.6852 97.79 0)
 			(hide yes)
 			(show_name no)
@@
 		)
 		(property "Datasheet" ""
-			(at 179.07 93.98 0)
+			(at 172.72 93.98 0)
 			(hide yes)
 			(show_name no)
@@
 		)
 		(property "Description" "Unpolarized capacitor"
-			(at 179.07 93.98 0)
+			(at 172.72 93.98 0)
 			(hide yes)
 			(show_name no)
@@
 	(symbol
 		(lib_id "Device:C")
-		(at 193.04 93.98 0)
+		(at 185.42 93.98 0)
 		(unit 1)
 		(body_style 1)
@@
 		(fields_autoplaced yes)
 		(property "Reference" "C7"
-			(at 196.85 92.7099 0)
+			(at 189.23 92.7099 0)
 			(show_name no)
 			(do_not_autoplace no)
@@
 		)
 		(property "Value" "100 nF"
-			(at 196.85 95.2499 0)
+			(at 189.23 95.2499 0)
 			(show_name no)
 			(do_not_autoplace no)
@@
 		)
 		(property "Footprint" ""
-			(at 194.0052 97.79 0)
+			(at 186.3852 97.79 0)
 			(hide yes)
 			(show_name no)
@@
 		)
 		(property "Datasheet" ""
-			(at 193.04 93.98 0)
+			(at 185.42 93.98 0)
 			(hide yes)
 			(show_name no)
@@
 		)
 		(property "Description" "Unpolarized capacitor"
-			(at 193.04 93.98 0)
-			(hide yes)
-			(show_name no)
+			(at 185.42 93.98 0)
+			(hide yes)
+			(show_name no)

Commit message: added footprints R and C and more
Parts:
- C5, C6, C7: footprint (none) -> Capacitor_SMD:C_0805_2012Metric_Pad1.18x1.45mm_HandSolder
- F2: footprint (none) -> Fuse:Fuse_0805_2012Metric_Pad1.15x1.40mm_HandSolder
Changed lines of the file:
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@@
 			)
 		)
-		(property "Footprint" ""
+		(property "Footprint" "Capacitor_SMD:C_0805_2012Metric_Pad1.18x1.45mm_HandSolder"
 			(at 173.6852 97.79 0)
 			(hide yes)
@@
 			)
 		)
-		(property "Footprint" ""
+		(property "Footprint" "Capacitor_SMD:C_0805_2012Metric_Pad1.18x1.45mm_HandSolder"
 			(at 186.3852 97.79 0)
 			(hide yes)
@@
 			)
 		)
-		(property "Footprint" ""
+		(property "Footprint" "Fuse:Fuse_0805_2012Metric_Pad1.15x1.40mm_HandSolder"
 			(at 83.82 91.948 90)
 			(hide yes)
@@
 			)
 		)
-		(property "Footprint" ""
+		(property "Footprint" "Capacitor_SMD:C_0805_2012Metric_Pad1.18x1.45mm_HandSolder"
 			(at 150.8252 97.79 0)
 			(hide yes)
