File: Servo_Power.kicad_sch (KiCad schematic)
At the start: 11 parts, among them J2 SERVO_BUCK_IN, J3 SERVO_BUCK_OUT, J4 Servo1, J5 Servo2, J6 Servo3, J7 Servo4, J8 Servo5

Commit message: added for 3v3 and 5v capacitors, resistors and induction footprints
Parts:
- C7: footprint Capacitor_SMD:C_0805_2012Metric_Pad1.18x1.45mm_HandSolder -> C1608X7R1H474K080AC:CAPC1608X90N
Changed lines of the file:
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@@
 			)
 		)
-		(property "Footprint" "Capacitor_SMD:C_0805_2012Metric_Pad1.18x1.45mm_HandSolder"
+		(property "Footprint" "C1608X7R1H474K080AC:CAPC1608X90N"
 			(at 186.3852 97.79 0)
 			(hide yes)
