File: imu.kicad_sch (KiCad schematic)
At the start: 14 parts, among them U2 BNO086, Y1 FC-135_32.7680KA-A0

Commit message: BNO086 switch SPI bus connection
Parts:
- removed R1: 0, symbol Device:R
- removed R2: DNI, symbol Device:R
- removed R3, R4: 2.2K, symbol Device:R
- removed R5: 10K, symbol Device:R
- added R10, R11, R8, R9: 10K, symbol Device:R
- added R12: 0R, symbol Device:R
Connections:
- net +3V3: now also R10.2, R11.2, R8.2, R9.2
- net BNO_CLKSEL0: now also R12.1
- net BNO_NRST: now also R11.1
- net GND: now also R12.2; no longer U2.5 (PS1), U2.6 (PS0/WAKE)
- net HOST_BOOTN: now also R8.1
- net HOST_MOSI: now reaches U2.17 (SA0/H_MOSI)
- net HOST_CSN: now reaches U2.18 (~{H_CS})
- net HOST_CSN: now also R10.1
- net HOST_SCL renamed HOST_SCLK
- net HOST_SDA renamed HOST_MISO
- new net BNO_WAKEUP/PS0: R9.1, U2.6 (PS0/WAKE)
- new net VDDIO: U2.5 (PS1)
Other:
- note added: "SPI connection"
- note removed: "I2C connection"

Commit message: connect BNO086 to MCU
Connections:
- net VDDIO is gone; now on net +3V3: U2.5 (PS1)
- net BNO_CLKSEL0: no longer names the net of R12.1, U2.10 (CLKSEL0)
Other:
- moved on the sheet: R12

Commit message: added footprints R and C and more
Parts:
- C10, C11, C12, C8, C9: footprint (none) -> Capacitor_SMD:C_0805_2012Metric_Pad1.18x1.45mm_HandSolder
- R10, R11, R12, R6, R7, R8, R9: footprint (none) -> Resistor_SMD:R_0805_2012Metric_Pad1.20x1.40mm_HandSolder
Changed lines of the file:
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@@
 			)
 		)
-		(property "Footprint" ""
+		(property "Footprint" "Capacitor_SMD:C_0805_2012Metric_Pad1.18x1.45mm_HandSolder"
 			(at 205.4352 59.69 0)
 			(hide yes)
@@
 			)
 		)
-		(property "Footprint" ""
+		(property "Footprint" "Capacitor_SMD:C_0805_2012Metric_Pad1.18x1.45mm_HandSolder"
 			(at 191.4652 59.69 0)
 			(hide yes)
@@
 			)
 		)
-		(property "Footprint" ""
+		(property "Footprint" "Resistor_SMD:R_0805_2012Metric_Pad1.20x1.40mm_HandSolder"
 			(at 184.15 94.488 90)
 			(hide yes)
@@
 			)
 		)
-		(property "Footprint" ""
+		(property "Footprint" "Resistor_SMD:R_0805_2012Metric_Pad1.20x1.40mm_HandSolder"
 			(at 180.34 80.772 90)
 			(hide yes)
@@
 			)
 		)
-		(property "Footprint" ""
+		(property "Footprint" "Capacitor_SMD:C_0805_2012Metric_Pad1.18x1.45mm_HandSolder"
 			(at 231.14 89.2048 0)
 			(hide yes)
@@
 			)
 		)
-		(property "Footprint" ""
+		(property "Footprint" "Resistor_SMD:R_0805_2012Metric_Pad1.20x1.40mm_HandSolder"
 			(at 107.442 100.33 90)
 			(hide yes)
@@
 			)
 		)
-		(property "Footprint" ""
+		(property "Footprint" "Resistor_SMD:R_0805_2012Metric_Pad1.20x1.40mm_HandSolder"
 			(at 56.642 88.9 90)
 			(hide yes)
@@
 			)
 		)
-		(property "Footprint" ""
+		(property "Footprint" "Capacitor_SMD:C_0805_2012Metric_Pad1.18x1.45mm_HandSolder"
 			(at 223.52 70.8152 0)
 			(hide yes)
@@
 			)
 		)
-		(property "Footprint" ""
+		(property "Footprint" "Capacitor_SMD:C_0805_2012Metric_Pad1.18x1.45mm_HandSolder"
 			(at 180.0352 100.33 0)
 			(hide yes)
@@
 			)
 		)
-		(property "Footprint" ""
+		(property "Footprint" "Resistor_SMD:R_0805_2012Metric_Pad1.20x1.40mm_HandSolder"
 			(at 84.582 95.25 90)
 			(hide yes)
@@
 			)
 		)
-		(property "Footprint" ""
+		(property "Footprint" "Resistor_SMD:R_0805_2012Metric_Pad1.20x1.40mm_HandSolder"
 			(at 180.34 78.232 90)
 			(hide yes)
@@
 			)
 		)
-		(property "Footprint" ""
+		(property "Footprint" "Resistor_SMD:R_0805_2012Metric_Pad1.20x1.40mm_HandSolder"
 			(at 98.552 97.79 90)
 			(hide yes)

Commit message: added footprints and connect usb33c MCU to power and VREF+ to REF3033
Parts:
- Y1: footprint FC-135_32.7680KA-A0:XTAL_FC-135_32.7680KA-A0 -> FC135:XTAL_FC-135_32.7680KA-A0
Changed lines of the file:
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@@
 			)
 		)
-		(property "Footprint" "FC-135_32.7680KA-A0:XTAL_FC-135_32.7680KA-A0"
+		(property "Footprint" "FC135:XTAL_FC-135_32.7680KA-A0"
 			(at 218.44 80.01 0)
 			(hide yes)
