File: 5v_buck.kicad_sch (KiCad schematic)
At the start: 11 parts, among them U5 LMR51430

Commit message: added for 3v3 and 5v capacitors, resistors and induction footprints
Parts:
- C24, C26: footprint (none) -> C1608X7R1H474K080AC:CAPC1608X90N
- C27, C28: footprint (none) -> C3216X7R1H475M160AC:CAPC3216X180N
- C29, C30, C31: footprint (none) -> C1206C105K5RACAUTO:CAPC3216X178N
- L1: footprint (none) -> Inductor_SMD:L_Coilcraft_XAL6060-XXX
- R3, R5: footprint (none) -> Resistor_SMD:R_0201_0603Metric
- U5: value LMR51430 -> LMR51430_5v
Changed lines of the file:
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@@
 			)
 		)
-		(property "Footprint" ""
+		(property "Footprint" "C1206C105K5RACAUTO:CAPC3216X178N"
 			(at 204.1652 106.68 0)
 			(hide yes)
@@
 			)
 		)
-		(property "Value" "LMR51430"
+		(property "Value" "LMR51430_5v"
 			(at 135.89 86.36 0)
 			(show_name no)
@@
 			)
 		)
-		(property "Footprint" ""
+		(property "Footprint" "C1206C105K5RACAUTO:CAPC3216X178N"
 			(at 192.7352 106.68 0)
 			(hide yes)
@@
 			)
 		)
-		(property "Footprint" ""
+		(property "Footprint" "C1206C105K5RACAUTO:CAPC3216X178N"
 			(at 113.9952 99.06 0)
 			(hide yes)
@@
 			)
 		)
-		(property "Footprint" ""
+		(property "Footprint" "Inductor_SMD:L_Coilcraft_XAL6060-XXX"
 			(at 172.72 96.52 0)
 			(hide yes)
@@
 			)
 		)
-		(property "Footprint" ""
+		(property "Footprint" "C3216X7R1H475M160AC:CAPC3216X180N"
 			(at 88.5952 99.06 0)
 			(hide yes)
@@
 			)
 		)
-		(property "Footprint" ""
+		(property "Footprint" "C1608X7R1H474K080AC:CAPC1608X90N"
 			(at 158.4452 96.52 0)
 			(hide yes)
@@
 			)
 		)
-		(property "Footprint" ""
+		(property "Footprint" "Resistor_SMD:R_0201_0603Metric"
 			(at 178.562 102.87 90)
 			(hide yes)
@@
 			)
 		)
-		(property "Footprint" ""
+		(property "Footprint" "Resistor_SMD:R_0201_0603Metric"
 			(at 178.562 113.03 90)
 			(hide yes)
@@
 			)
 		)
-		(property "Footprint" ""
+		(property "Footprint" "C3216X7R1H475M160AC:CAPC3216X180N"
 			(at 101.2952 99.06 0)
 			(hide yes)
@@
 			)
 		)
-		(property "Footprint" ""
+		(property "Footprint" "C1608X7R1H474K080AC:CAPC1608X90N"
 			(at 74.6252 99.06 0)
 			(hide yes)
