File: pesokbot_board.kicad_sch (KiCad schematic)
At the start: 0 parts

Commit message: added 3v3 buck converter
Other:
- added sheet 3V3_BUCK (3v3_buck.kicad_sch)
Changed lines of the file:
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@@
+	)
+	(sheet
+		(at 180.34 96.52)
+		(size 12.7 5.08)
+		(exclude_from_sim no)
+		(in_bom yes)
+		(on_board yes)
+		(dnp no)
+		(fields_autoplaced yes)
+		(stroke
+			(width 0.1524)
+			(type solid)
+		)
+		(fill
+			(color 0 0 0 0)
+		)
+		(property "Sheetname" "3V3_BUCK"
+			(at 180.34 95.8084 0)
+			(show_name no)
+			(do_not_autoplace no)
+			(effects
+				(font
+					(size 1.27 1.27)
+				)
+				(justify left bottom)
+			)
+		)
+		(property "Sheetfile" "3v3_buck.kicad_sch"
+			(at 180.34 102.1846 0)
+			(show_name no)
+			(do_not_autoplace no)
+			(effects
+				(font
+					(size 1.27 1.27)
+				)
+				(justify left top)
+			)
+		)
+		(instances
+			(project "pesokbot_board"
+				(path "/3b0b46ed-3ce3-4874-97d9-085fc63ec69d"
+					(page "10")
+				)
+			)
+		)
 	)
 	(sheet

Commit message: change vbat_prot footprint and added pwrmux for 3v3 ubs_mcu connector
Other:
- added sheet TPS2121RUXR_pwrmux (TPS2121RUXR_pwrmux.kicad_sch)
Changed lines of the file:
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@@
+	)
+	(sheet
+		(at 202.565 96.52)
+		(size 12.7 6.35)
+		(exclude_from_sim no)
+		(in_bom yes)
+		(on_board yes)
+		(dnp no)
+		(fields_autoplaced yes)
+		(stroke
+			(width 0.1524)
+			(type solid)
+		)
+		(fill
+			(color 0 0 0 0)
+		)
+		(property "Sheetname" "TPS2121RUXR_pwrmux"
+			(at 202.565 95.8084 0)
+			(show_name no)
+			(do_not_autoplace no)
+			(effects
+				(font
+					(size 1.27 1.27)
+				)
+				(justify left bottom)
+			)
+		)
+		(property "Sheetfile" "TPS2121RUXR_pwrmux.kicad_sch"
+			(at 202.565 103.4546 0)
+			(show_name no)
+			(do_not_autoplace no)
+			(effects
+				(font
+					(size 1.27 1.27)
+				)
+				(justify left top)
+			)
+		)
+		(instances
+			(project "pesokbot_board"
+				(path "/3b0b46ed-3ce3-4874-97d9-085fc63ec69d"
+					(page "11")
+				)
+			)
+		)
 	)
 	(sheet

Commit message: added LTC4412 powerpath component for usb mcu power
Other:
- sheet TPS2121RUXR_pwrmux renamed LTC4412_pwrpath
- sheet LTC4412_pwrpath: file TPS2121RUXR_pwrmux.kicad_sch -> LTC4412_pwrpath.kicad_sch
Changed lines of the file:
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@@
 			(color 0 0 0 0)
 		)
-		(property "Sheetname" "TPS2121RUXR_pwrmux"
+		(property "Sheetname" "LTC4412_pwrpath"
 			(at 202.565 95.8084 0)
 			(show_name no)
@@
 			)
 		)
-		(property "Sheetfile" "TPS2121RUXR_pwrmux.kicad_sch"
+		(property "Sheetfile" "LTC4412_pwrpath.kicad_sch"
 			(at 202.565 103.4546 0)
 			(show_name no)
