File: LTC4412_pwrpath.kicad_sch (KiCad schematic)
At the start: 1 part, among them U8 LTC4412xS6

Commit message: delete bad files
Parts:
- removed U8: LTC4412xS6, Package_TO_SOT_SMD:TSOT-23-6, symbol Power_Management:LTC4412xS6
- added C38: 22µF, C1608X7R1H474K080AC:CAPC1608X90N, symbol C1608X7R1H474K080AC:C1608X7R1H474K080AC
- added C39: 100nF, C1608X7R1H474K080AC:CAPC1608X90N, symbol C1608X7R1H474K080AC:C1608X7R1H474K080AC
- added Q3, Q4: AO4407A, Package_SO:SOIC-8_3.9x4.9mm_P1.27mm, symbol Transistor_FET:AO4407A
- added R13: 470K, symbol Device:R
- added U9: LTC4412xS6, Package_TO_SOT_SMD:TSOT-23-6, symbol Power_Management:LTC4412xS6
Connections:
- net GND: now also C38.2, C39.2, U9.2 (GND), U9.3 (CTL)
- net USB_MCU_VBUS: now also Q4.[5-8] (Drain)
- net VBAT_PROT: now also C39.1, Q3.[5-8] (Drain), U9.1 (VIN)
- new net +VIN_3V3_MUX: C38.1, Q3.[1-3] (Source), Q4.[1-3] (Source), R13.2, U9.6 (SENSE)
- new net AUXILIARY_GATE: Q4.4 (Gate), R13.1, U9.4 (STAT)
- new net PRIMARY_GATE: Q3.4 (Gate), U9.5 (GATE)
