File: pesokbot_board.kicad_pcb (KiCad board)
At the start: 4 copper layers, 80 x 60 mm, 65 parts, among them J1 J_BAT_3S2P, J10 Conn_02x06_Odd_Even, J11 Conn_02x06_Odd_Even, J12 Conn_02x06_Odd_Even, J13 Conn_02x06_Odd_Even, J14 Conn_02x06_Odd_Even, J15 Conn_02x06_Odd_Even, J16 Conn_02x06_Odd_Even, J17 Conn_02x06_Odd_Even, J18 Conn_02x06_Odd_Even, J19 Conn_02x06_Odd_Even, J20 Conn_02x06_Odd_Even, J21 Conn_02x06_Odd_Even, J9 Conn_02x06_Odd_Even, P1 USB_C_Plug_USB2.0, P2 USB_C_Plug_USB2.0, Q1 SQJQ100E, U1 LM74700, U2 BNO086, U3 STM32H743ZIT6, U4 REF3033, Y1 FC-135_32.7680KA-A0

Commit message: added 5v buck converter and place JST PH connectors
Parts:
- P1: value USB_C_Plug_USB2.0 -> USB-CDC
- P2: value USB_C_Plug_USB2.0 -> USB-MCU
- moved J21 283.6 mm to (183.1, 74.0)
- moved J13 263.3 mm to (193.1, 140.7), turned to 180 degrees
- moved J20 252.2 mm to (176.2, 140.7), turned to 180 degrees
- moved J14 249.0 mm to (166.2, 74.0)
- moved J17 231.8 mm to (159.2, 140.7), turned to 180 degrees
- moved J11 226.8 mm to (149.2, 74.0)
- moved J15 213.4 mm to (142.3, 140.7), turned to 180 degrees
- moved J19 201.2 mm to (125.5, 140.7), turned to 180 degrees
- moved J16 188.1 mm to (104.0, 95.5), turned to 90 degrees
- moved J18 187.1 mm to (104.0, 112.3), turned to 90 degrees
- moved J12 174.5 mm to (104.0, 129.2), turned to 90 degrees
- moved REF** 32.1 mm to (203.5, 139.7)
- moved REF** 28.5 mm to (203.5, 74.5)
- moved REF** 14.7 mm to (105.0, 139.7)
- moved J1 6.49 mm to (-17.5, 67.5)
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Other:
- board size 80 x 60 mm -> 108.5 x 74.7 mm

Commit message: added for 3v3 and 5v capacitors, resistors and induction footprints
Parts:
- removed P1: USB-CDC, Connector_USB:USB_C_Receptacle_HRO_TYPE-C-31-M-12
- removed P2: USB-MCU, Connector_USB:USB_C_Receptacle_HRO_TYPE-C-31-M-12
- added 5.1K3: R, Resistor_SMD:R_0805_2012Metric_Pad1.20x1.40mm_HandSolder, F.Cu at (-120.6, 219.6)
- added 5.1K4: R, Resistor_SMD:R_0805_2012Metric_Pad1.20x1.40mm_HandSolder, F.Cu at (-120.6, 222.5)
- added 5.1K5: R, Resistor_SMD:R_0805_2012Metric_Pad1.20x1.40mm_HandSolder, F.Cu at (-164.0, 205.3)
- added 5.1K6: R, Resistor_SMD:R_0805_2012Metric_Pad1.20x1.40mm_HandSolder, F.Cu at (-164.0, 208.2)
- added C24: 100 nF, C1608X7R1H474K080AC:CAPC1608X90N, F.Cu at (-153.1, 221.3)
- added C25: 10nF, Capacitor_SMD:C_0805_2012Metric_Pad1.18x1.45mm_HandSolder, F.Cu at (-145.8, 223.7)
- added C26: 100 nF, C1608X7R1H474K080AC:CAPC1608X90N, F.Cu at (-153.1, 223.8)
- added C27: 4.7uF, C3216X7R1H475M160AC:CAPC3216X180N, F.Cu at (-157.9, 221.7)
- added C28: 4.7uF, C3216X7R1H475M160AC:CAPC3216X180N, F.Cu at (-157.9, 225.1)
- added C29: 22uF, C1206C105K5RACAUTO:CAPC3216X178N, F.Cu at (-163.6, 213.4)
- added C30: 22uF, C1206C105K5RACAUTO:CAPC3216X178N, F.Cu at (-163.6, 216.8)
- added C31: 22uF, C1206C105K5RACAUTO:CAPC3216X178N, F.Cu at (-163.6, 220.1)
- added C32: 4.7µF, C3216X7R1H475M160AC:CAPC3216X180N, F.Cu at (-141.8, 195.0)
- added C33: 4.7µF, C3216X7R1H475M160AC:CAPC3216X180N, F.Cu at (-141.8, 198.4)
- added C34: 0.1µF, C1608X7R1H474K080AC:CAPC1608X90N, F.Cu at (-142.6, 205.9)
- added C35: 22µF, C1206C105K5RACAUTO:CAPC3216X178N, F.Cu at (-149.9, 203.3)
- added C36: 22µF, C1206C105K5RACAUTO:CAPC3216X178N, F.Cu at (-149.9, 206.7)
- added C37: 0.1µF, C1608X7R1H474K080AC:CAPC1608X90N, F.Cu at (-142.6, 208.4)
- added J22: USB-MCU, Connector_USB:USB_C_Receptacle_HRO_TYPE-C-31-M-12, F.Cu at (-77.9, 176.4)
- added J23: USB-CDC, Connector_USB:USB_C_Receptacle_HRO_TYPE-C-31-M-12, F.Cu at (-98.6, 174.8)
- added L1: 6.8uH, Inductor_SMD:L_Coilcraft_XAL6060-XXX, F.Cu at (-115.4, 164.9)
- added L2: 5.6µH, Inductor_SMD:L_Coilcraft_XAL6060-XXX, F.Cu at (-127.6, 164.8)
- added R14: 22.1K, Resistor_SMD:R_0201_0603Metric, F.Cu at (-139.4, 205.6)
- added R15: 100K, Resistor_SMD:R_0201_0603Metric, F.Cu at (-139.4, 207.3)
- added R3: 100K, Resistor_SMD:R_0201_0603Metric, F.Cu at (-151.4, 212.6)
- added R4: 1M, Resistor_SMD:R_0805_2012Metric_Pad1.20x1.40mm_HandSolder, F.Cu at (-127.0, 219.6)
- added R5: 13.7K, Resistor_SMD:R_0201_0603Metric, F.Cu at (-151.4, 214.3)
- added U5: LMR51430_5v, Package_TO_SOT_SMD:SOT-23-6, F.Cu at (-128.4, 204.7)
- added U6: LMR51430_3v3, Package_TO_SOT_SMD:SOT-23-6, F.Cu at (-111.4, 206.6)
- C1, C13, C17, C19, C2, C20, C22, C7: footprint Capacitor_SMD:C_0805_2012Metric_Pad1.18x1.45mm_HandSolder -> C1608X7R1H474K080AC:CAPC1608X90N
Connections:
- F2 pad 1: unconnected-(F2-Pad1) -> VBAT_PROT

Commit message: change vbat_prot footprint and added pwrmux for 3v3 ubs_mcu connector
Parts:
- J1: footprint Connector_JST:JST_EH_B2B-EH-A_1x02_P2.50mm_Vertical -> TerminalBlock_Phoenix:TerminalBlock_Phoenix_MKDS-1,5-2-5.08_1x02_P5.08mm_Horizontal
- moved L2 309.6 mm to (172.8, 89.7)
- moved J1 224.5 mm to (203.0, 109.9), turned to 90 degrees
- moved C13 19.3 mm to (128.0, 132.0)
- moved C15 19.3 mm to (131.0, 132.0)
- moved C16 19.3 mm to (134.0, 132.0)
- moved C19 19.3 mm to (137.3, 132.0)
- moved C17 19.3 mm to (116.8, 131.9)
- moved C18 19.3 mm to (119.8, 131.9)
- moved R1 19.3 mm to (122.5, 131.9)
- moved R7 15.3 mm to (166.2, 112.3)
- moved R10 14.1 mm to (169.9, 106.8)
- moved R6 11.6 mm to (160.8, 108.9)
- moved C14 9.68 mm to (117.2, 93.4)
- moved U2 9.60 mm to (154.0, 107.3)
- moved U3 9.15 mm to (128.9, 107.3)

Commit message: delete bad files
Parts:
- added C38: 22µF, C1608X7R1H474K080AC:CAPC1608X90N, F.Cu at (-168.3, 158.7)
- added C39: 100nF, C1608X7R1H474K080AC:CAPC1608X90N, F.Cu at (-168.3, 161.1)
- added Q3: AO4407A, Package_SO:SOIC-8_3.9x4.9mm_P1.27mm, F.Cu at (-174.5, 156.2)
- added Q4: AO4407A, Package_SO:SOIC-8_3.9x4.9mm_P1.27mm, F.Cu at (-174.5, 162.7)
- added U9: LTC4412xS6, Package_TO_SOT_SMD:TSOT-23-6, F.Cu at (-167.7, 155.2)
Connections:
- C32 pad 1: +5V_MAIN -> +VBAT_MUX
- C33 pad 1: +5V_MAIN -> +VBAT_MUX
- C37 pad 1: +5V_MAIN -> +VBAT_MUX
- J22 pad A4: unconnected-(J22-VBUS-PadA4)_2 -> USB_MCU_VBUS
- J22 pad A9: unconnected-(J22-VBUS-PadA4) -> USB_MCU_VBUS
- J22 pad B4: unconnected-(J22-VBUS-PadA4)_3 -> USB_MCU_VBUS
- J22 pad B9: unconnected-(J22-VBUS-PadA4)_1 -> USB_MCU_VBUS
- U6 pad 3: +5V_MAIN -> +VBAT_MUX
- U6 pad 5: +5V_MAIN -> +VBAT_MUX
